File: Hardware/Qwiic Joystick_Eagle/Qwiic Joystick.sch (EAGLE design)
At the start: 26 parts, among them J6 AVR_SPI_PROG_3X2TESTPOINTS, U2 ATTINY85

Commit message: updating buzzard labels to include fatter arrows
Parts:
- added H5, H6: STAND-OFF, SparkFun-Hardware:STAND-OFF
Other:
- note added: "Kevin Kuwata, Andy England"
- note added: "Vin: 2.7-5.5V"
- note added: "v10"
- note removed: "Kevin Kuwata"
- note removed: "v01"
Changed lines of the file:
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@@
 <part name="H4" library="SparkFun-Hardware" deviceset="STAND-OFF" device=""/>
 <part name="U2" library="SparkFun-IC-Microcontroller" deviceset="ATTINY85" device=""/>
+<part name="H5" library="SparkFun-Hardware" deviceset="STAND-OFF" device=""/>
+<part name="H6" library="SparkFun-Hardware" deviceset="STAND-OFF" device=""/>
 </parts>
 <sheets>
@@
 <plain>
 <text x="166.6748" y="11.3284" size="2.54" layer="94" font="vector">Nick Poole</text>
-<text x="237.744" y="7.366" size="2.54" layer="94" font="vector">v01</text>
+<text x="237.744" y="7.366" size="2.54" layer="94" font="vector">v10</text>
 <text x="209.9818" y="165.9382" size="1.778" layer="97" font="vector">Power
 Indicator</text>
-<text x="169.9768" y="7.0104" size="2.54" layer="94" font="vector">Kevin Kuwata</text>
+<text x="169.9768" y="7.0104" size="2.54" layer="94" font="vector">Kevin Kuwata, Andy England</text>
 <text x="108.966" y="51.308" size="2.032" layer="97" font="vector" rot="R90" align="top-left">I2C Port</text>
 <text x="96.52" y="154.94" size="1.778" layer="97" font="vector">Pogo Programmer</text>
@@
 <text x="149.86" y="104.14" size="2.54" layer="97" font="vector">Joystick</text>
 <text x="2.54" y="104.14" size="2.54" layer="97" font="vector">I2C Connections</text>
+<text x="2.54" y="177.8" size="1.27" layer="97" font="vector">Vin: 2.7-5.5V</text>
 </plain>
 <instances>
@@
 <instance part="LOGO1" gate="G$1" x="169.672" y="44.958"/>
 <instance part="U$1" gate="G$1" x="190.5" y="35.56"/>
-<instance part="J6" gate="G$1" x="104.14" y="142.24">
+<instance part="J6" gate="G$1" x="104.14" y="142.24" smashed="yes">
+<attribute name="NAME" x="99.06" y="147.828" size="1.778" layer="95" font="vector"/>
 <attribute name="NAME" x="99.06" y="147.828" size="1.778" layer="95" font="vector"/>
 </instance>
@@
 <attribute name="NAME" x="33.02" y="152.908" size="1.778" layer="95" font="vector"/>
 </instance>
+<instance part="H5" gate="G$1" x="231.14" y="30.48"/>
+<instance part="H6" gate="G$1" x="231.14" y="27.94"/>
 </instances>
 <busses>

Commit message: updating resistor values
Parts:
- R1, R7: value 2.2K -> 2.2k; device SparkFun-Resistors:4.7KOHM-0603-1/10W-1% -> SparkFun-Resistors:2.2KOHM-0603-1/10W-1%
- R8: value 10K -> 10k; device SparkFun-Resistors:330OHM-0603-1/10W-1% -> SparkFun-Resistors:10KOHM-0603-1/10W-1%
Changed lines of the file:
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@@
 <part name="H2" library="SparkFun-Hardware" deviceset="STAND-OFF" device=""/>
 <part name="GND3" library="SparkFun-PowerSymbols" deviceset="GND" device=""/>
-<part name="R1" library="SparkFun-Resistors" deviceset="4.7KOHM" device="-0603-1/10W-1%" value="2.2K"/>
-<part name="R7" library="SparkFun-Resistors" deviceset="4.7KOHM" device="-0603-1/10W-1%" value="2.2K"/>
+<part name="R1" library="SparkFun-Resistors" deviceset="2.2KOHM" device="-0603-1/10W-1%" value="2.2k"/>
+<part name="R7" library="SparkFun-Resistors" deviceset="2.2KOHM" device="-0603-1/10W-1%" value="2.2k"/>
 <part name="JP7" library="SparkFun-Jumpers" deviceset="JUMPER-SMT_3_2-NC_TRACE" device="_NO-SILK" value="JUMPER-SMT_3_2-NC_TRACE_NO-SILK"/>
 <part name="SUPPLY9" library="SparkFun-PowerSymbols" deviceset="3.3V" device=""/>
-<part name="R8" library="SparkFun-Resistors" deviceset="330OHM" device="-0603-1/10W-1%" value="10K"/>
+<part name="R8" library="SparkFun-Resistors" deviceset="10KOHM" device="-0603-1/10W-1%" value="10k"/>
 <part name="SUPPLY6" library="SparkFun-PowerSymbols" deviceset="3.3V" device=""/>
 <part name="LOGO2" library="SparkFun-Aesthetics" deviceset="REVISION" device=""/>
